File: pcb/eidon-tracker/eidon-tracker.kicad_pcb (KiCad board)
At the start: 2 copper layers, 29.5 x 24.2 mm, 11 parts, among them SW1 SW_SPDT, SW2 SW_Push, U1 XIAO-ESP32-C6, U2 GY-BNO085

Commit message: fix(pcb): adds corrected BOM for incorrect LED resistor value
Parts:
- R3: value 1.8k -> 1k
Changed lines of the file:
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@@
 			)
 		)
-		(property "Description" ""
-			(at 0.022323 -0.012888 90)
+		(property "Description" "XIAO-ESP32C6 MCU Module"
+			(at 0 0 0)
 			(unlocked yes)
 			(layer "F.Fab")
@@
 			(effects
 				(font
-					(size 1.27 1.27)
+					(size 1 1)
 					(thickness 0.15)
 				)
@@
 			)
 		)
-		(property "Description" "XIAO-ESP32C6 MCU Module"
-			(at 0 0 0)
-			(unlocked yes)
-			(layer "F.Fab")
-			(hide yes)
-			(effects
-				(font
-					(size 1 1)
-					(thickness 0.15)
-				)
-			)
-		)
 		(sheetname "/")
 		(sheetfile "eidon-tracker.kicad_sch")
@@
 			)
 		)
-		(property "Value" "1.8k"
+		(property "Value" "1k"
 			(at 0 0 0)
 			(layer "B.Fab")
@@
 					(thickness 0.15)
 				)
+				(justify mirror)
+			)
+		)
+		(property "Supplier & Ref" "LCSC C95781; Digi-Key 311-1.00KCRCT-ND"
+			(at 0 0 0)
+			(unlocked yes)
+			(layer "B.Fab")
+			(hide yes)
+			(effects
+				(font
+					(size 1 1)
+					(thickness 0.15)
+				)
+				(justify mirror)
+			)
+		)
+		(property "Manufacturer Part Number (MPN)" "Yageo RC0805FR-071KL"
+			(at 0 0 0)
+			(unlocked yes)
+			(layer "B.Fab")
+			(hide yes)
+			(effects
+				(font
+					(size 1 1)
+					(thickness 0.15)
+				)
