File: pcb/eidon-tracker/eidon-tracker.kicad_sch (KiCad schematic)
At the start: 9 parts, among them SW1 SW_SPDT, SW2 SW_Push, U1 XIAO-ESP32-C6, U2 GY-BNO085

Commit message: fix(pcb): adds corrected BOM for incorrect LED resistor value
Parts:
- SW2: Supplier & Ref Mouser 688-SKRKACE010 -> LCSC SKRKAEE020; Mouser 688-SKRKACE010
Changed lines of the file:
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@@
 			)
 		)
-		(property "Supplier & Ref" "Mouser 688-SKRKACE010"
+		(property "Supplier & Ref" "LCSC SKRKAEE020; Mouser 688-SKRKACE010"
 			(at 196.85 137.16 0)
 			(effects
