File: pcb/eidon-tracker-v4/eidon-tracker.kicad_sch (KiCad schematic)
At the start: 11 parts, among them SW1 SW_SPDT, U1 XIAO-ESP32-C6, U2 BNO085

Commit message: fix(pcb): corrects component placement so not too close to edge per jlcpcb rejection feedback
Parts:
- removed R3, R5: 2.2k, Resistor_SMD:R_0805_2012Metric, symbol Device:R
- added C1, C2: 22pF, Capacitor_SMD:C_0603_1608Metric, symbol Device:C
- added C3, C4, C5: 100nF, Capacitor_SMD:C_0603_1608Metric, symbol Device:C
- added R6, R7: 10k, Resistor_SMD:R_0805_2012Metric, symbol Device:R
- added X1: 32.768KHz, Crystal:Crystal_SMD_3215-2Pin_3.2x1.5mm, symbol Device:Crystal
- U1: footprint XIAO-ESP32-C6 -> eidon-tracker:XIAO-ESP32C6-SMD; now in the parts list
- U2: footprint LGA-28_CEV -> eidon-tracker:BNO085
- renumbered R6 to R3, R7 to R5
Connections:
- net GND: now also U2.18 (H_CSN), U2.5 (PS1), U2.6 (PS0/WAKE), C1.1, C2.1, C3.1, C4.1, C5.1
- net RST: now also R6.1; no longer U1.6 (GPIO23_D5_SCL)
- net VCC: now also C4.2, C5.2, R6.2, R7.2
- net at U2.15 (ENV_SCL): no longer R4.1
- net XOUT: now reaches U2.26 (XOUT32/CLKSEL1)
- net XOUT: now also C2.2, X1.2
- net XIN: now reaches U2.27 (XIN32)
- net XIN: now also C1.2, X1.1
- net CAP: now reaches U2.9 (CAP)
- net CAP: now also C3.2
- net BOOT: no longer names the net of U1.23 (BOOT)
- net CS: no longer names the net of U1.8 (GPIO17_D7_RX)
- net CS: no longer U2.18 (H_CSN)
- net MISO renamed SDA
- net SDA: now also R4.1
- net MOSI renamed SDO
- net SDO: now also R7.1
- net PS0: no longer names the net of U1.3 (GPIO2_A2_D2)
- net PS0: no longer U2.6 (PS0/WAKE)
- net PS1: no longer names the net of U1.4 (GPIO21_D3)
- net PS1: no longer U2.5 (PS1)
- net SCK renamed SCL
- no-connect marks 10 -> 17
Other:
- note removed: "BUTTON"
- note removed: "LED"
- moved on the sheet: R3, R5, U2
